File: hardware/OpenAIO.kicad_pcb (KiCad board)
At the start: 8 copper layers, 35 x 35 mm, 285 parts, among them J1 OpenDrone-Core, J10 5V, J12 5V, J13 5V, J14 5V, J15 5V, J16 5V, J17 5V, J18 5V, J19 5V, J2 Conn_Coaxial_Small, J20 5V, J21 5V, J22 5V, J23 5V, J24 5V, J25 5V, J26 5V, J27 5V, J28 5V, J29 5V, J3 5V, J30 5V, J31 5V, J32 5V, J35 5V, J36 5V, J37 5V, J38 5V, J4 5V, J5 5V, J6 5V, J8 5V, J9 5V, Q1 DOY180N03T, Q10 DOY180N03T, Q11 DOY180N03T, Q12 DOY180N03T, Q13 DOY180N03T, Q14 DOY180N03T, Q15 DOY180N03T, Q16 DOY180N03T, Q17 DOY180N03T, Q18 DOY180N03T, Q19 DOY180N03T, Q2 DOY180N03T, Q20 DOY180N03T, Q21 DOY180N03T, Q22 DOY180N03T, Q23 DOY180N03T, Q24 DOY180N03T, Q3 DOY180N03T, Q4 DOY180N03T, Q5 DOY180N03T, Q6 DOY180N03T, Q7 DOY180N03T, Q8 DOY180N03T, Q9 DOY180N03T, T1 0900PC16J0042001E, U1 AIO_outline, U10 SM06B-SRSS-TB(LF)(SN), U11 AT32F421G8U7, U12 NSG2065Q, U13 AT32F421G8U7, U14 NSG2065Q, U15 AT32F421G8U7, U16 NSG2065Q, U17 AT32F421G8U7, U18 NSG2065Q, U19 INA186A3IDCKR, U22 TS2306A 240GF MSM 9_C2976675, U3 LR1121IMLTRT, U4 ESP32-C3, U5 RFX2401C, U6 TLV75533PDQNR, U7 SKY13373-460LF, U8 LMR51430YFDDCR, U9 LMR51430YFDDCR, X1 CJ17-400001010B20

Commit message: Routing cheat sheet on Cmts.User: vias, keys, escapes, limits
Replaces the prose how-to beside the outline with a keyword table.

Co-Authored-By: Claude Opus 5.5 <noreply@anthropic.com>
Other:
- board text added: "ROUTING CHEAT SHEET - 8L HDI 1+6+1 - NextPCB LAYERS L1 parts | L2 GND | L3 sig | L4 PWR | L5 PWR | L6 sig | L7 GND | L8 parts VIA SIZE SPAN KEY micro 0.25/0.10 L1-L2 L8-L7 Ctrl+V buried 0.40/0.20 (PWR 0.45/0.25) L2-L7 Alt+Shift+V through 0.40/0.20 V layer pair preset "Buried L2-L7" Shift+V cycle ESCAPE GND pin pad > micro > L2 done signal pad > micro > buried > L3/L6 stagger 0.25 c-c power micro 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"
- board text removed: "HDI 1+6+1 NextPCB. L1 parts | L2 GND | L3 sig | L4 PWR | L5 PWR | L6 sig | L7 GND | L8 parts Vias: laser 0.25/0.10 L1-L2, L8-L7 | buried L2-L7 and through 0.40/0.20 default (power 0.45/0.25, 0.50/0.30) Route (X). V = through via. Ctrl+V = microvia. Alt+Shift+V = blind/buried via (uses active layer pair). Layer pair presets are preloaded (Route > Set Layer Pair): "Buried L2-L7" In1.Cu/In6.Cu, "Out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"
Changed lines of the file:
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@@
 		)
 	)
-	(gr_text "HDI 1+6+1 NextPCB. L1 parts | L2 GND | L3 sig | L4 PWR | L5 PWR | L6 sig | L7 GND | L8 parts\nVias: laser 0.25/0.10 L1-L2, L8-L7 | buried L2-L7 and through 0.40/0.20 default (power 0.45/0.25, 0.50/0.30)\nRoute (X). V = through via. Ctrl+V = microvia. Alt+Shift+V = blind/buried via (uses active layer pair).\nLayer pair presets are preloaded (Route > Set Layer Pair): \"Buried L2-L7\" In1.Cu/In6.Cu, \"Outer F-B\"; Shift+V cycles.\nAlt+< = select layer then place blind/buried via. After placing, E on the via: check type and layers.\nSizes: Board Setup > Design Rules > Pre-defined Sizes; pick via size in the toolbar before placing.\nGND pin: pad > Ctrl+V microvia into the pad > done (L2 is GND). Bottom: pad > Ctrl+V to In6.\nSignal: pad > Ctrl+V to In1 > Alt+Shift+V buried 0.25 mm beside it (lands overlap, no L2 track) > route on In2/In5.\nPower: pad > microvias > buried vias staggered > In3/In4 plane connects through the buried via.\nNever stack a microvia on a buried via; stagger 0.25 mm c-c. Never microvia L1-L3 (skip via).\nFine pitch (<= 0.5 mm): microvia in pad, filled and capped (IPC-4761 VII). Buried vias are resin filled.\nPower and phase: arrays of microvias and buried vias, 0.20 mm same-net hole spacing.\nRF: no vias on RF nets, 0.105 mm CPWG gap 0.15 on L1/L8, L2/L7 solid below.\nRun DRC after each block; \"blind via\" errors mean Alt+Shift+V picked the wrong type."
+	(gr_text "ROUTING CHEAT SHEET  -  8L HDI 1+6+1  -  NextPCB\nLAYERS   L1 parts | L2 GND | L3 sig | L4 PWR | L5 PWR | L6 sig | L7 GND | L8 parts\n\nVIA          SIZE                     SPAN        KEY\nmicro        0.25/0.10                L1-L2 L8-L7 Ctrl+V\nburied       0.40/0.20  (PWR 0.45/0.25) L2-L7       Alt+Shift+V\nthrough      0.40/0.20   V\nlayer pair   preset \"Buried L2-L7\"                Shift+V cycle\n\nESCAPE\nGND pin      pad > micro > L2              done\nsignal       pad > micro > buried > L3/L6  stagger 0.25 c-c\npower        micro array > buried array > L4/L5\nfine pitch   micro in pad (filled + capped)\n\nNEVER\nmicro on buried (stacked)   micro L1-L3   via on RF net\ntracks on L2/L7             2 oz copper (forces 5/5 mil)\n\nWIDTHS\nmin track 0.089 (3.5 mil)   RF 50R 0.105 gap 0.15   USB 90R 0.12/0.12\n\nCHECK\nE on via = type + layers    DRC after each block    B = refill zones"
 		(at 96 43.5 0)
 		(layer "Cmts.User")
 		(effects
 			(font
-				(size 1 1)
-				(line_spacing 1.4)
-				(thickness 0.15)
+				(size 0.8 0.8)
+				(thickness 0.12)
 			)
 			(justify left top)
@@
 	)
 	(gr_text "OpenAIO STACKUP 1.6 mm, 8 layer HDI 1+6+1, all copper 1 oz (0.035), mask 0.015\nLayer | KiCad | Use                                   | Dielectric below (mm)\nL1 | F.Cu   | parts, RF, USB, power loops             | 1080 0.077\nL2 | In1.Cu | GND plane, no tracks (type power)       | 2116 0.125\nL3 | In2.Cu | signals + +BATT zone (mixed)           | core 0.330\nL4 | In3.Cu | +4v5/+3V3/+5V_USB zones + signals       | 2116+2313 0.228\nL5 | In4.Cu | +5V/+3V3 zones + signals                | core 0.330\nL6 | In5.Cu | signals + +10V/+BATT zones              | 2116 0.125\nL7 | In6.Cu | GND plane, no tracks (type power)       | 1080 0.077\nL8 | B.Cu   | parts, RF, power\nVIA | span | drill/pad (mm)\nLaser micro | F.Cu-In1.Cu, In6.Cu-B.Cu | 0.10/0.25\nBuried | In1.Cu-In6.Cu | 0.20/0.40 (power 0.25/0.45)\nThrough | F.Cu-B.Cu | 0.20/0.40 default, 0.25/0.45, 0.30/0.50\nBlind mechanical: not allowed (DRC rule)"
-		(at 96 73 0)
+		(at 96 77.52947 0)
 		(layer "Cmts.User")
 		(effects

Commit message: Allow a microvia stacked on a same-net buried via; Mac keys in the cheat sheet
Owner decision 2026-10-13: stacking allowed at the HDI II (Rank 2) price.
Rule: same-net micro/buried hole spacing 0 (stacked or staggered);
holes_co_located is already a warning on this board.
Cheat sheet: Cmd+V microvia, Opt+Shift+V buried, Opt+V layer pick.

Co-Authored-By: Claude Opus 5.5 <noreply@anthropic.com>
Other:
- board text added: "ROUTING CHEAT SHEET - 8L HDI 1+6+1 - NextPCB - macOS keys LAYERS L1 parts | L2 GND | L3 sig | L4 PWR | L5 PWR | L6 sig | L7 GND | L8 parts VIA SIZE SPAN KEY (Mac) micro 0.25/0.10 L1-L2 L8-L7 Cmd+V buried 0.40/0.20 (PWR 0.45/0.25) L2-L7 Opt+Shift+V through 0.40/0.20 L1-L8 V pick layer Select Layer box, then via Opt+V label check 1-2 / 7-8 micro | 2-7 buried | 1-8 through ESCAPE (stacked allowed, o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"
- board text removed: "ROUTING CHEAT SHEET - 8L HDI 1+6+1 - NextPCB LAYERS L1 parts | L2 GND | L3 sig | L4 PWR | L5 PWR | L6 sig | L7 GND | L8 parts VIA SIZE SPAN KEY micro 0.25/0.10 L1-L2 L8-L7 Ctrl+V buried 0.40/0.20 (PWR 0.45/0.25) L2-L7 Alt+Shift+V through 0.40/0.20 V layer pair preset "Buried L2-L7" Shift+V cycle ESCAPE GND pin pad > micro > L2 done signal pad > micro > buried > L3/L6 stagger 0.25 c-c power micro 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"
Changed lines of the file:
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@@
 		)
 	)
-	(gr_text "ROUTING CHEAT SHEET  -  8L HDI 1+6+1  -  NextPCB\nLAYERS   L1 parts | L2 GND | L3 sig | L4 PWR | L5 PWR | L6 sig | L7 GND | L8 parts\n\nVIA          SIZE                     SPAN        KEY\nmicro        0.25/0.10                L1-L2 L8-L7 Ctrl+V\nburied       0.40/0.20  (PWR 0.45/0.25) L2-L7       Alt+Shift+V\nthrough      0.40/0.20   V\nlayer pair   preset \"Buried L2-L7\"                Shift+V cycle\n\nESCAPE\nGND pin      pad > micro > L2              done\nsignal       pad > micro > buried > L3/L6  stagger 0.25 c-c\npower        micro array > buried array > L4/L5\nfine pitch   micro in pad (filled + capped)\n\nNEVER\nmicro on buried (stacked)   micro L1-L3   via on RF net\ntracks on L2/L7             2 oz copper (forces 5/5 mil)\n\nWIDTHS\nmin track 0.089 (3.5 mil)   RF 50R 0.105 gap 0.15   USB 90R 0.12/0.12\n\nCHECK\nE on via = type + layers    DRC after each block    B = refill zones"
+	(gr_text "ROUTING CHEAT SHEET  -  8L HDI 1+6+1  -  NextPCB  -  macOS keys\nLAYERS   L1 parts | L2 GND | L3 sig | L4 PWR | L5 PWR | L6 sig | L7 GND | L8 parts\n\nVIA          SIZE                     SPAN         KEY (Mac)\nmicro        0.25/0.10                L1-L2 L8-L7  Cmd+V\nburied       0.40/0.20  (PWR 0.45/0.25) L2-L7        Opt+Shift+V\nthrough      0.40/0.20               L1-L8        V\npick layer   Select Layer box, then via            Opt+V\nlabel check  1-2 / 7-8 micro | 2-7 buried | 1-8 through\n\nESCAPE (stacked allowed, order = HDI Rank 2)\nGND pin      pad > Cmd+V > L2                 done\nsignal       pad > Cmd+V > Opt+Shift+V same spot > L3/L6\npower        stacked micro+buried array > L4/L5\nfine pitch   micro in pad (filled + capped)\noptional     stagger buried 0.25 c-c (lands overlap)\n\nNEVER\nmicro on micro   micro L1-L3   via on RF net   tracks on L2/L7   2 oz copper\n\nWIDTHS\nmin track 0.089 (3.5 mil)   RF 50R 0.105 gap 0.15   USB 90R 0.12/0.12\n\nCHECK\nE on via = type + layers   DRC per block   B = refill zones\n\"holes co-located\" warning on a stack = expected"
 		(at 96 43.5 0)
 		(layer "Cmts.User")
