File: hardware/OpenAIO.kicad_pcb (KiCad board)
At the start: 8 copper layers, 35 x 35 mm, 285 parts, among them J1 OpenDrone-Core, J10 5V, J12 5V, J13 5V, J14 5V, J15 5V, J16 5V, J17 5V, J18 5V, J19 5V, J2 Conn_Coaxial_Small, J20 5V, J21 5V, J22 5V, J23 5V, J24 5V, J25 5V, J26 5V, J27 5V, J28 5V, J29 5V, J3 5V, J30 5V, J31 5V, J32 5V, J35 5V, J36 5V, J37 5V, J38 5V, J4 5V, J5 5V, J6 5V, J8 5V, J9 5V, Q1 DOY180N03T, Q10 DOY180N03T, Q11 DOY180N03T, Q12 DOY180N03T, Q13 DOY180N03T, Q14 DOY180N03T, Q15 DOY180N03T, Q16 DOY180N03T, Q17 DOY180N03T, Q18 DOY180N03T, Q19 DOY180N03T, Q2 DOY180N03T, Q20 DOY180N03T, Q21 DOY180N03T, Q22 DOY180N03T, Q23 DOY180N03T, Q24 DOY180N03T, Q3 DOY180N03T, Q4 DOY180N03T, Q5 DOY180N03T, Q6 DOY180N03T, Q7 DOY180N03T, Q8 DOY180N03T, Q9 DOY180N03T, T1 0900PC16J0042001E, U1 AIO_outline, U10 SM06B-SRSS-TB(LF)(SN), U11 AT32F421G8U7, U12 NSG2065Q, U13 AT32F421G8U7, U14 NSG2065Q, U15 AT32F421G8U7, U16 NSG2065Q, U17 AT32F421G8U7, U18 NSG2065Q, U19 INA186A3IDCKR, U22 TS2306A 240GF MSM 9_C2976675, U3 LR1121IMLTRT, U4 ESP32-C3, U5 RFX2401C, U6 TLV75533PDQNR, U7 SKY13373-460LF, U8 LMR51430YFDDCR, U9 LMR51430YFDDCR, X1 CJ17-400001010B20

Commit message: Cheat sheet: via keys match the remapped user.hotkeys (V micro, Shift+V buried)
Co-Authored-By: Claude Opus 5.5 <noreply@anthropic.com>
Other:
- board text added: "ROUTING CHEAT SHEET - 8L HDI 1+6+1 - NextPCB - keys from user.hotkeys (Cmd+V = paste) LAYERS L1 parts | L2 GND | L3 sig | L4 PWR | L5 PWR | L6 sig | L7 GND | L8 parts VIA SIZE SPAN KEY (Mac) micro 0.25/0.10 L1-L2 L8-L7 V (while routing) buried 0.38/0.20 (all classes) L2-L7 Shift+V through 0.38/0.20 L1-L8 Cmd+Opt+Shift+V pick layer Opt+V (blind; "via pass" converts it) label check 1-2 / 7-8 micro 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"
- board text removed: "ROUTING CHEAT SHEET - 8L HDI 1+6+1 - NextPCB - macOS keys LAYERS L1 parts | L2 GND | L3 sig | L4 PWR | L5 PWR | L6 sig | L7 GND | L8 parts VIA SIZE SPAN KEY (Mac) micro 0.25/0.10 L1-L2 L8-L7 Cmd+V buried 0.38/0.20 (all classes) L2-L7 Opt+Shift+V through 0.38/0.20 L1-L8 V pick layer Select Layer box, then via Opt+V label check 1-2 / 7-8 micro | 2-7 buried | 1-8 through ESCAPE (stacked allowed, ord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"
Changed lines of the file:
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@@
 		)
 	)
-	(gr_text "ROUTING CHEAT SHEET  -  8L HDI 1+6+1  -  NextPCB  -  macOS keys\nLAYERS   L1 parts | L2 GND | L3 sig | L4 PWR | L5 PWR | L6 sig | L7 GND | L8 parts\n\nVIA          SIZE                     SPAN         KEY (Mac)\nmicro        0.25/0.10                L1-L2 L8-L7  Cmd+V\nburied       0.38/0.20  (all classes) L2-L7        Opt+Shift+V\nthrough      0.38/0.20               L1-L8        V\npick layer   Select Layer box, then via            Opt+V\nlabel check  1-2 / 7-8 micro | 2-7 buried | 1-8 through\n\nESCAPE (stacked allowed, order = HDI Rank 2)\nGND pin      pad > Cmd+V > L2                 done\nsignal       pad > Cmd+V > Opt+Shift+V same spot > L3/L6\npower        stacked micro+buried array > L4/L5\nfine pitch   micro in pad (filled + capped)\noptional     stagger buried 0.25 c-c (lands overlap)\n\nNEVER\nmicro on micro   micro L1-L3   via on RF net   tracks on L2/L7   2 oz copper\n\nWIDTHS\nmin track 0.089 (3.5 mil)   RF 50R 0.105 gap 0.15   USB 90R 0.12/0.12\n\nCHECK\nE on via = type + layers   DRC per block   B = refill zones\n\"holes co-located\" warning on a stack = expected"
+	(gr_text "ROUTING CHEAT SHEET  -  8L HDI 1+6+1  -  NextPCB  -  keys from user.hotkeys (Cmd+V = paste)\nLAYERS   L1 parts | L2 GND | L3 sig | L4 PWR | L5 PWR | L6 sig | L7 GND | L8 parts\n\nVIA          SIZE                     SPAN         KEY (Mac)\nmicro        0.25/0.10                L1-L2 L8-L7  V (while routing)\nburied       0.38/0.20  (all classes) L2-L7        Shift+V\nthrough      0.38/0.20               L1-L8        Cmd+Opt+Shift+V\npick layer   Opt+V (blind; \"via pass\" converts it)\nlabel check  1-2 / 7-8 micro | 2-7 buried | 1-8 through\n\nESCAPE (stacked allowed, order = HDI Rank 2)\nGND pin      pad > V > L2                 done\nsignal       pad > V > Shift+V same spot > L3/L6\npower        stacked micro+buried array > L4/L5\nfine pitch   micro in pad (filled + capped)\noptional     stagger buried 0.25 c-c (lands overlap)\n\nNEVER\nmicro on micro   micro L1-L3   via on RF net   tracks on L2/L7   2 oz copper\n\nWIDTHS\nmin track 0.089 (3.5 mil)   RF 50R 0.105 gap 0.15   USB 90R 0.12/0.12\n\nCHECK\nE on via = type + layers   DRC per block   B = refill zones\n\"holes co-located\" warning on a stack = expected"
 		(at 96 43.5 0)
 		(layer "Cmts.User")
