File: hardware/OpenAIO.kicad_sch (KiCad schematic)
At the start: 15 parts, among them J1 OpenDrone-Core, U1 AIO_outline, U19 INA186A3IDCKR

Commit message: schematic review: USB D+/D- swap, bulk cap parts, VTX UART, EN series R, density cuts, ERC cleanup, docs (#24)
Items 1, 2, 3, 5, 8, 9, 10, 11, 12, 13, 14 (partial), 17, 18, 19, 20, 21, 22, 23, 6.
Edits are structured s-expression edits re-saved by kicad-cli sch upgrade.

Co-authored-by: Stan <stan@openaio.local>
Co-authored-by: Claude Opus 5.5 <noreply@anthropic.com>
Parts:
- removed C94: 100nF, Capacitor_SMD:C_0201_0603Metric, symbol ESCLibrary:GRM033R61C104KE84D
- removed R95: 1k, 4in1ESC:R_0201_0603Metric, symbol ESCLibrary:0201_1kR
- C84: footprint Capacitor_SMD:C_0402_1005Metric -> Capacitor_SMD:C_0201_0603Metric; Cost 0.003257 -> 0.025; LCSC C7500381 -> C76935; MPN CC0402KRX7R6BB105 -> GRM033R61A105ME44D; Manufacturer YAGEO -> Murata Electronics
- R93, R94: footprint Capacitor_SMD:C_0201_0603Metric -> Resistor_SMD:R_0201_0603Metric
Connections:
- net Pads/UART1_TX is gone; now on net Pads/PIOUART0_RX: J1.39 (PIOUART0_RX)
- net CURR: now also U19.6 (OUT)
- net D+: now also J1.22 (D+); no longer J1.15 (D-)
- net D-: now also J1.15 (D-); no longer J1.22 (D+)
- net Pads/PIOUART0_RX: no longer J1.48 (UART0_TX)
- net Pads/PIOUART0_TX: now also J1.40 (PIOUART0_TX); no longer J1.49 (UART0_RX)
- net Pads/UART0_RX: now also J1.49 (UART0_RX); no longer J1.31 (PIOUART1_TX)
- net Pads/UART0_TX: now also J1.48 (UART0_TX); no longer J1.40 (PIOUART0_TX)
- net Pads/UART1_RX renamed Pads/PIOUART1_RX
- no-connect marks 5 -> 6
Other:
- sheet ESC1 ports: added MotorA, MotorB, MotorC; removed A, B, C
- sheet ESC2 ports: added MotorA, MotorB, MotorC; removed A, B, C
- sheet ESC3 ports: added MotorA, MotorB, MotorC; removed A, B, C
- sheet ESC4 ports: added MotorA, MotorB, MotorC; removed A, B, C
- sheet Pads ports: added PIOUART1_RX; removed UART1_RX, UART1_TX
