File: hardware/esc_channel.kicad_sch (KiCad schematic)
At the start: 39 parts, among them Q1 DOY180N03T, Q2 DOY180N03T, Q3 DOY180N03T, Q4 DOY180N03T, Q5 DOY180N03T, Q6 DOY180N03T, U11 AT32F421G8U7, U12 NSG2065Q

Commit message: schematic review: USB D+/D- swap, bulk cap parts, VTX UART, EN series R, density cuts, ERC cleanup, docs (#24)
Items 1, 2, 3, 5, 8, 9, 10, 11, 12, 13, 14 (partial), 17, 18, 19, 20, 21, 22, 23, 6.
Edits are structured s-expression edits re-saved by kicad-cli sch upgrade.

Co-authored-by: Stan <stan@openaio.local>
Co-authored-by: Claude Opus 5.5 <noreply@anthropic.com>
Parts:
- removed R19, R20: 10k, Resistor_SMD:R_0201_0603Metric, symbol ESCLibrary:0201_10kR
- C70: renamed from C50; value C -> 4.7uF 50v; LCSC (none) -> C98192; MPN (none) -> CL21A475KBQNNNE; Manufacturer (none) -> Samsung Electro-Mechanics
- C71: renamed from C51; value C -> 4.7uF 50v; LCSC (none) -> C98192; MPN (none) -> CL21A475KBQNNNE; Manufacturer (none) -> Samsung Electro-Mechanics
- C72: renamed from C52; value C -> 4.7uF 50v; LCSC (none) -> C98192; MPN (none) -> CL21A475KBQNNNE; Manufacturer (none) -> Samsung Electro-Mechanics
- renumbered C47 to C35, C48 to C39, C44 to C78, C45 to C79, C43 to C80, C46 to C83, C49 to C88, Q1 to Q19, Q2 to Q20, Q3 to Q21, Q4 to Q22, Q5 to Q23, Q6 to Q24, R17 to R55, R18 to R56, R21 to R59, R23 to R60, R24 to R61, R25 to R62, R26 to R63, R27 to R64, R28 to R65, R29 to R66, R30 to R67, R31 to R68, R32 to R69, R33 to R70, R34 to R71, R35 to R72, R22 to R77, TP3 to TP7, TP4 to TP8, U11 to U10, U12 to U11
Connections:
- net A renamed MotorA
- net B renamed MotorB
- net C renamed MotorC
- no-connect marks 14 -> 15
