File: hardware/esc_channel.kicad_sch (KiCad schematic)
At the start: 39 parts, among them Q1 DOY180N03T, Q2 DOY180N03T, Q3 DOY180N03T, Q4 DOY180N03T, Q5 DOY180N03T, Q6 DOY180N03T, U11 AT32F421G8U7, U12 NSG2065Q

Commit message: One board: Base + Core merged on the 8L HDI stackup, replaces the OpenFC-Core module layout (#25)
* Base fully routed (recovered from KiCad local history, 2026-08-22)

The finished Base route was never committed: the last Base commit (ce0aa59)
had 57 unconnected. Recovered from hardware/.history snapshot 55d048e
(last save 2026-08-22 15:03), on top of ce0aa59.

DRC (kicad-cli 10):
- Base: 0 unconnected, 0 shorts, 6 errors (3 x U23 own pad-to-pad
  clearance, USB1 NPTH: 1 clearance + 2 annular width), 111 warnings
- Core: 0 unconnected, 0 errors

Co-Authored-By: Claude Opus 5.5 <noreply@anthropic.com>

* Power: +10V buck always on with battery, 10V_ENABLE removed

CIRCUIT_REVIEW B1: the LMR51430 +10V buck U3 (NSG2065Q gate drive and VTX power) was enabled by RP2354A GPIO27 over LGA pad 1 with no pull, so firmware or a Betaflight PINIO could cut ESC gate drive, and on USB-only power a high GPIO27 drove EN with VIN = 0, which the LMR51430 datasheet forbids. U3 EN is now tied to +BATT exactly like U4 (datasheet: EN may be tied to VIN; no parts added). Base: U3.5 keeps its B.Cu stub and through via, re-netted to +BATT so the via lands in the +BATT planes; the In2 run, the via and the F.Cu stub to J90 pad 1 are removed. Core: the GPIO27 route to J91 pad 1 is removed. LGA pad 1 and GPIO27 are free (no-connect); the root marker TP14 of the old net is dropped. Boards saved by pcbnew 10.0.6 without zone refill; the "Tokyo" silkscreen render caches were re-rendered with a substitute font (Tokyo not installed here).

Co-Authored-By: Claude Opus 5.5 <noreply@anthropic.com>
Claude-Session: https://claude.ai/code/session_01KTp3FLjVXfXdWrkmr6af7d

* Review of the split Core/Base design, NextPCB rules, re-route plan

Circuit review against datasheets, layout review (LGA interface, DC power
solver, noise, density, assembly, DRC) with the scripts that produced every
number, NextPCB fab and assembly limits with sources, and the plan with the
decisions taken for the re-route.

Co-Author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
Parts:
- C35: renamed from C47; footprint Capacitor_SMD:C_0402_WIDE -> lib:C_0402_WIDE; symbol ESCLibrary:GRM033R61C104KE84D -> lib:GRM033R61C104KE84D; Manufacturer (none) -> Samsung Electro-Mechanics
- C39: renamed from C48; footprint Capacitor_SMD:C_0402_WIDE -> lib:C_0402_WIDE; symbol ESCLibrary:GRM033R61C104KE84D -> lib:GRM033R61C104KE84D; Manufacturer (none) -> Samsung Electro-Mechanics
- C78: renamed from C44; footprint Capacitor_SMD:C_0201_0603Metric -> lib:C_0201_0603Metric; symbol ESCLibrary:GRM033R61C104KE84D -> lib:GRM033R61C104KE84D; Manufacturer (none) -> Murata Electronics
- C79: renamed from C45; footprint Capacitor_SMD:C_0201_0603Metric -> lib:C_0201_0603Metric; symbol ESCLibrary:GRM033R61C104KE84D -> lib:GRM033R61C104KE84D; Manufacturer (none) -> Murata Electronics
- C80: renamed from C43; footprint Capacitor_SMD:C_0201_0603Metric -> lib:C_0201_0603Metric; symbol ESCLibrary:GRM033R61C104KE84D -> lib:GRM033R61C104KE84D; Manufacturer (none) -> Murata Electronics
- C83: renamed from C46; footprint Capacitor_SMD:C_0402_WIDE -> lib:C_0402_WIDE; symbol ESCLibrary:GRM033R61C104KE84D -> lib:GRM033R61C104KE84D; Manufacturer (none) -> Samsung Electro-Mechanics
- C88: renamed from C49; footprint Capacitor_SMD:C_0201_0603Metric -> lib:C_0201_0603Metric; symbol ESCLibrary:GRM033R61C104KE84D -> lib:GRM033R61C104KE84D; Manufacturer (none) -> Murata Electronics
- C96: renamed from C50; value C -> 4.7uF 50v; footprint Capacitor_SMD:C_0805_2012Metric -> lib:C_0805_2012Metric; LCSC (none) -> C98192; MPN (none) -> CL21A475KBQNNNE; Manufacturer (none) -> Samsung Electro-Mechanics
- C97: renamed from C51; value C -> 4.7uF 50v; footprint Capacitor_SMD:C_0805_2012Metric -> lib:C_0805_2012Metric; LCSC (none) -> C98192; MPN (none) -> CL21A475KBQNNNE; Manufacturer (none) -> Samsung Electro-Mechanics
- C98: renamed from C52; value C -> 4.7uF 50v; footprint Capacitor_SMD:C_0805_2012Metric -> lib:C_0805_2012Metric; LCSC (none) -> C98192; MPN (none) -> CL21A475KBQNNNE; Manufacturer (none) -> Samsung Electro-Mechanics
- Q19: renamed from Q1; footprint Package_SON:Diodes_PowerDI3333-8 -> lib:DOY180N03T_TDFN3333-8; symbol PCM_Transistor_MOSFET_AKL:2N6660 -> lib:2N6660; Manufacturer (none) -> DOINGTER
- Q20: renamed from Q2; footprint Package_SON:Diodes_PowerDI3333-8 -> lib:DOY180N03T_TDFN3333-8; symbol PCM_Transistor_MOSFET_AKL:2N6660 -> lib:2N6660; Manufacturer (none) -> DOINGTER
- Q21: renamed from Q3; footprint Package_SON:Diodes_PowerDI3333-8 -> lib:DOY180N03T_TDFN3333-8; symbol PCM_Transistor_MOSFET_AKL:2N6660 -> lib:2N6660; Manufacturer (none) -> DOINGTER
- Q22: renamed from Q4; footprint Package_SON:Diodes_PowerDI3333-8 -> lib:DOY180N03T_TDFN3333-8; symbol PCM_Transistor_MOSFET_AKL:2N6660 -> lib:2N6660; Manufacturer (none) -> DOINGTER
- Q23: renamed from Q5; footprint Package_SON:Diodes_PowerDI3333-8 -> lib:DOY180N03T_TDFN3333-8; symbol PCM_Transistor_MOSFET_AKL:2N6660 -> lib:2N6660; Manufacturer (none) -> DOINGTER
- Q24: renamed from Q6; footprint Package_SON:Diodes_PowerDI3333-8 -> lib:DOY180N03T_TDFN3333-8; symbol PCM_Transistor_MOSFET_AKL:2N6660 -> lib:2N6660; Manufacturer (none) -> DOINGTER
- R55: renamed from R17; footprint Resistor_SMD:R_0201_0603Metric -> lib:R_0201_0603Metric; symbol PCM_Resistor_AKL:R_0402 -> lib:R_0402; Manufacturer (none) -> UNI-ROYAL
- R56: renamed from R18; footprint Resistor_SMD:R_0201_0603Metric -> lib:R_0201_0603Metric; symbol PCM_Resistor_AKL:R_0402 -> lib:R_0402; Manufacturer (none) -> UNI-ROYAL
- R57: renamed from R19; footprint Resistor_SMD:R_0201_0603Metric -> lib:R_0201_0603Metric; symbol ESCLibrary:0201_10kR -> lib:0201_10kR; Manufacturer (none) -> YAGEO
- R58: renamed from R20; footprint Resistor_SMD:R_0201_0603Metric -> lib:R_0201_0603Metric; symbol ESCLibrary:0201_10kR -> lib:0201_10kR; Manufacturer (none) -> YAGEO
- R59: renamed from R21; footprint Resistor_SMD:R_0201_0603Metric -> lib:R_0201_0603Metric; symbol ESCLibrary:0201_220R -> lib:0201_220R; Manufacturer (none) -> YAGEO
- R60: renamed from R23; footprint Resistor_SMD:R_0201_0603Metric -> lib:R_0201_0603Metric; symbol PCM_Resistor_AKL:R_0402 -> lib:R_0402; Manufacturer (none) -> UNI-ROYAL
- R61: renamed from R24; footprint Resistor_SMD:R_0201_0603Metric -> lib:R_0201_0603Metric; symbol PCM_Resistor_AKL:R_0402 -> lib:R_0402; Manufacturer (none) -> UNI-ROYAL
- R62: renamed from R25; footprint Resistor_SMD:R_0201_0603Metric -> lib:R_0201_0603Metric; symbol PCM_Resistor_AKL:R_0402 -> lib:R_0402; Manufacturer (none) -> UNI-ROYAL
- R63: renamed from R26; footprint Resistor_SMD:R_0201_0603Metric -> lib:R_0201_0603Metric; symbol PCM_Resistor_AKL:R_0402 -> lib:R_0402; Manufacturer (none) -> UNI-ROYAL
- R64: renamed from R27; footprint Resistor_SMD:R_0201_0603Metric -> lib:R_0201_0603Metric; symbol ESCLibrary:0201_10kR -> lib:0201_10kR; Manufacturer (none) -> YAGEO
- R65: renamed from R28; footprint Resistor_SMD:R_0201_0603Metric -> lib:R_0201_0603Metric; symbol ESCLibrary:0201_1kR -> lib:0201_1kR; Manufacturer (none) -> UNI-ROYAL
- R66: renamed from R29; footprint Resistor_SMD:R_0201_0603Metric -> lib:R_0201_0603Metric; symbol ESCLibrary:0201_10kR -> lib:0201_10kR; Manufacturer (none) -> YAGEO
- R67: renamed from R30; footprint Resistor_SMD:R_0201_0603Metric -> lib:R_0201_0603Metric; symbol ESCLibrary:0201_10kR -> lib:0201_10kR; Manufacturer (none) -> YAGEO
- R68: renamed from R31; footprint Resistor_SMD:R_0201_0603Metric -> lib:R_0201_0603Metric; symbol ESCLibrary:0201_1kR -> lib:0201_1kR; Manufacturer (none) -> UNI-ROYAL
- R69: renamed from R32; footprint Resistor_SMD:R_0201_0603Metric -> lib:R_0201_0603Metric; symbol ESCLibrary:0201_10kR -> lib:0201_10kR; Manufacturer (none) -> YAGEO
- R70: renamed from R33; footprint Resistor_SMD:R_0201_0603Metric -> lib:R_0201_0603Metric; symbol ESCLibrary:0201_10kR -> lib:0201_10kR; Manufacturer (none) -> YAGEO
- R71: renamed from R34; footprint Resistor_SMD:R_0201_0603Metric -> lib:R_0201_0603Metric; symbol ESCLibrary:0201_1kR -> lib:0201_1kR; Manufacturer (none) -> UNI-ROYAL
- R72: renamed from R35; footprint Resistor_SMD:R_0201_0603Metric -> lib:R_0201_0603Metric; symbol ESCLibrary:0201_10kR -> lib:0201_10kR; Manufacturer (none) -> YAGEO
- R77: renamed from R22; footprint Resistor_SMD:R_0201_0603Metric -> lib:R_0201_0603Metric; Manufacturer (none) -> YAGEO
- TP7: renamed from TP3; footprint TestPoint:TestPoint_Pad_D1.0mm -> lib:TestPoint_Pad_D1.0mm
- TP8: renamed from TP4; footprint TestPoint:TestPoint_Pad_D1.0mm -> lib:TestPoint_Pad_D1.0mm
- U10: renamed from U11; footprint 4in1ESC:QFN-28_L4.0-W4.0-P0.40-TL-EP2.4 -> lib:QFN-28_L4.0-W4.0-P0.40-TL-EP2.4; symbol ESCLibrary:AT32F421G8U7 -> lib:AT32F421G8U7
- U11: renamed from U12; footprint 4in1ESC:QFN-24_L4.0-W4.0-P0.50-TL-EP2.8 -> lib:QFN-24_L4.0-W4.0-P0.50-TL-EP2.8; symbol components:NSG2065Q -> lib:NSG2065Q; Manufacturer (none) -> NSIC
Connections:
- net +3V3 renamed +3V3_ESC
Other:
- title: (none) -> ESC channel
