File: hardware/esp32c3_lr1121_mono.kicad_sch (KiCad schematic)
At the start: 57 parts, among them J2 Conn_Coaxial_Small, T1 0900PC16J0042001E, U22 TS2306A 240GF MSM 9_C2976675, U3 LR1121IMLTRT, U4 ESP32-C3, U5 RFX2401C, U6 TLV75533PDQNR, U7 SKY13373-460LF, X1 CJ17-400001010B20

Commit message: schematic review: USB D+/D- swap, bulk cap parts, VTX UART, EN series R, density cuts, ERC cleanup, docs (#24)
Items 1, 2, 3, 5, 8, 9, 10, 11, 12, 13, 14 (partial), 17, 18, 19, 20, 21, 22, 23, 6.
Edits are structured s-expression edits re-saved by kicad-cli sch upgrade.

Co-authored-by: Stan <stan@openaio.local>
Co-authored-by: Claude Opus 5.5 <noreply@anthropic.com>
Parts:
- removed U22: TS2306A 240GF MSM 9_C2976675, lib:SW-SMD_4P-L3.0-W2.0-P0.85-LS3.5, symbol lib:TS2306A240GFMSM9_C2976675
- added J39: BOOT, OpenDrone:SolderPad_1.0x0.8mm, symbol Connector_Generic:Conn_01x01
- C23, C31: MPN (none) -> CL05A106MQ5NUNC; Manufacturer (none) -> Samsung Electro-Mechanics
- C26, C30: MPN (none) -> GRM033R61A105ME44D; Manufacturer (none) -> Murata Electronics
- U1: renamed from U4; value ESP32-C3 -> ESP32-C3FH4; LCSC (none) -> C2858491; MPN (none) -> ESP32-C3FH4; Manufacturer (none) -> Espressif Systems
- U5: renamed from U7; LCSC (none) -> C150853; MPN (none) -> SKY13373-460LF; Manufacturer (none) -> Skyworks Solutions
- U6: MPN (none) -> TLV75533PDQNR; Manufacturer (none) -> Texas Instruments
- renumbered C4 to C1, C9 to C11, C2 to C12, C3 to C13, C7 to C14, C10 to C15, C12 to C16, C5 to C19, C17 to C2, C15 to C20, C24 to C21, C29 to C22, C28 to C23, C32 to C24, C13 to C25, C18 to C26, C19 to C27, C21 to C28, C22 to C29, C8 to C3, C25 to C30, C27 to C31, C20 to C4, C14 to C5, C16 to C6, C6 to C7, C11 to C9, J2 to J1, L3 to L1, L1 to L2, L2 to L3, L5 to L4, L4 to L5, R7 to R1, R4 to R2, R5 to R3, R6 to R4, R10 to R5, R3 to R6, R8 to R7, R9 to R8, U5 to U4
Connections:
- net ELRS_BOOT: now also J39.1 (Pin_1)
