File: hardware/fc_pads.kicad_sch (KiCad schematic)
At the start: 37 parts, among them J10 5V, J11 5V, J12 5V, J13 5V, J14 5V, J15 5V, J16 5V, J17 5V, J18 5V, J19 5V, J20 5V, J21 5V, J22 5V, J23 5V, J24 5V, J25 5V, J26 5V, J27 5V, J28 5V, J29 5V, J3 5V, J30 5V, J31 5V, J32 5V, J33 5V, J34 5V, J35 5V, J36 5V, J37 5V, J38 5V, J4 5V, J5 5V, J6 5V, J7 5V, J8 5V, J9 5V, U10 SM06B-SRSS-TB(LF)(SN)

Commit message: schematic review: USB D+/D- swap, bulk cap parts, VTX UART, EN series R, density cuts, ERC cleanup, docs (#24)
Items 1, 2, 3, 5, 8, 9, 10, 11, 12, 13, 14 (partial), 17, 18, 19, 20, 21, 22, 23, 6.
Edits are structured s-expression edits re-saved by kicad-cli sch upgrade.

Co-authored-by: Stan <stan@openaio.local>
Co-authored-by: Claude Opus 5.5 <noreply@anthropic.com>
Parts:
- removed J10, J11, J15, J17, J20, J33, J4, J6, J7: 5V, lib:small_pad, symbol Connector_Generic:Conn_01x01
Connections:
- net UART1_TX is gone; now on net PIOUART0_RX: J12.1 (Pin_1)
- net PIOUART0_RX: now also J35.1 (Pin_1), U10.4; no longer J32.1 (Pin_1)
- net PIOUART0_TX: now also J36.1 (Pin_1), U10.3; no longer J31.1 (Pin_1)
- net UART0_RX: now also J31.1 (Pin_1); no longer J35.1 (Pin_1), U10.4
- net UART0_TX: now also J32.1 (Pin_1); no longer J36.1 (Pin_1), U10.3
- net UART1_RX renamed PIOUART1_RX
