File: hardware/fc_pads.kicad_sch (KiCad schematic)
At the start: 37 parts, among them J10 5V, J11 5V, J12 5V, J13 5V, J14 5V, J15 5V, J16 5V, J17 5V, J18 5V, J19 5V, J20 5V, J21 5V, J22 5V, J23 5V, J24 5V, J25 5V, J26 5V, J27 5V, J28 5V, J29 5V, J3 5V, J30 5V, J31 5V, J32 5V, J33 5V, J34 5V, J35 5V, J36 5V, J37 5V, J38 5V, J4 5V, J5 5V, J6 5V, J7 5V, J8 5V, J9 5V, U10 SM06B-SRSS-TB(LF)(SN)

Commit message: One board: Base + Core merged on the 8L HDI stackup, replaces the OpenFC-Core module layout (#25)
* Base fully routed (recovered from KiCad local history, 2026-08-22)

The finished Base route was never committed: the last Base commit (ce0aa59)
had 57 unconnected. Recovered from hardware/.history snapshot 55d048e
(last save 2026-08-22 15:03), on top of ce0aa59.

DRC (kicad-cli 10):
- Base: 0 unconnected, 0 shorts, 6 errors (3 x U23 own pad-to-pad
  clearance, USB1 NPTH: 1 clearance + 2 annular width), 111 warnings
- Core: 0 unconnected, 0 errors

Co-Authored-By: Claude Opus 5.5 <noreply@anthropic.com>

* Power: +10V buck always on with battery, 10V_ENABLE removed

CIRCUIT_REVIEW B1: the LMR51430 +10V buck U3 (NSG2065Q gate drive and VTX power) was enabled by RP2354A GPIO27 over LGA pad 1 with no pull, so firmware or a Betaflight PINIO could cut ESC gate drive, and on USB-only power a high GPIO27 drove EN with VIN = 0, which the LMR51430 datasheet forbids. U3 EN is now tied to +BATT exactly like U4 (datasheet: EN may be tied to VIN; no parts added). Base: U3.5 keeps its B.Cu stub and through via, re-netted to +BATT so the via lands in the +BATT planes; the In2 run, the via and the F.Cu stub to J90 pad 1 are removed. Core: the GPIO27 route to J91 pad 1 is removed. LGA pad 1 and GPIO27 are free (no-connect); the root marker TP14 of the old net is dropped. Boards saved by pcbnew 10.0.6 without zone refill; the "Tokyo" silkscreen render caches were re-rendered with a substitute font (Tokyo not installed here).

Co-Authored-By: Claude Opus 5.5 <noreply@anthropic.com>
Claude-Session: https://claude.ai/code/session_01KTp3FLjVXfXdWrkmr6af7d

* Review of the split Core/Base design, NextPCB rules, re-route plan

Circuit review against datasheets, layout review (LGA interface, DC power
solver, noise, density, assembly, DRC) with the scripts that produced every
number, NextPCB fab and assembly limits with sources, and the plan with the
decisions taken for the re-route.

Co-Author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
Parts:
- added C114, C115: 100n, lib:C_0201_0603Metric, symbol Device:C
- added D10: SDM02U30LP3-7B, lib:X3-DFN0603-2_L0.6-W0.3-RD, symbol lib:SDM02U30LP3-7B
- added J23: SCL, lib:small_pad, symbol Connector_Generic:Conn_01x01
- added J26: SDA, lib:small_pad, symbol Connector_Generic:Conn_01x01
- added J30: 5V, lib:small_pad, symbol Connector_Generic:Conn_01x01
- added J34: GND, lib:small_pad, symbol Connector_Generic:Conn_01x01
- added U28: DPS368XTSA1, lib:LGA-8_L2.5-W2.0-P0.65-TR_DPS368, symbol lib:DPS368XTSA1
- J17: renamed from J5; value 5V -> GND
- J18: renamed from J6; value 5V -> GND
- J19: renamed from J7; value 5V -> ADC2
- J20: renamed from J9; value 5V -> LED
- J21: renamed from J10; value 5V -> LED
- J22: renamed from J11; value 5V -> GND
- J27: renamed from J17; value 5V -> GND
- J28: renamed from J18; value 5V -> GND
- J29: renamed from J19; value 5V -> BUZ-
- J31: renamed from J20; value 5V -> LED
- J32: renamed from J21; value 5V -> LED
- J33: renamed from J22; value 5V -> BUZ+
- J35: renamed from J23; value 5V -> GND
- J38: renamed from J25; value 5V -> CAM
- J39: renamed from J26; value 5V -> VTX
- J40: renamed from J27; value 5V -> GND
- J41: renamed from J28; value 5V -> 10V; footprint lib:small_pad -> lib:SolderPad_1.2x1.2mm
- J42: renamed from J29; value 5V -> 4V5
- J43: renamed from J30; value 5V -> GND
- J44: renamed from J31; value 5V -> PIO_TX0
- J45: renamed from J32; value 5V -> PIO_RX0
- J46: renamed from J33; value 5V -> NC
- J47: renamed from J34; value 5V -> NC
- J48: renamed from J35; value 5V -> RX0
- J49: renamed from J36; value 5V -> TX0
- J50: renamed from J37; value 5V -> GND
- J51: renamed from J38; value 5V -> GND; footprint lib:small_pad -> lib:SolderPad_1.2x1.2mm
- J52: renamed from J14; value 5V -> 4V5
- J53: renamed from J13; value 5V -> GND
- J54: renamed from J12; value 5V -> TX1
- J55: renamed from J8; value 5V -> RX1
- renumbered J3 to J15, J4 to J16, J15 to J24, J16 to J25, J24 to J37, U10 to U12
Connections:
- net +10V: no longer J51.1 (Pin_1)
- net +5V: now also D10.1 (C), J30.1 (Pin_1)
- net BUZZER-: now also D10.2 (A)
- net GND: now also J51.1 (Pin_1), C114.2, C115.2, J34.1 (Pin_1), U28.1 (GND), U28.5 (SDO), U28.7 (GND)
- net UART1_RX: no longer J46.1 (Pin_1), U12.6
- net PIOUART0_RX renamed PU0RX
- net PU0RX: now also J46.1 (Pin_1), U12.6
- new net +3.3V: C114.1, C115.1, U28.2 (CSB), U28.6 (VDDIO), U28.8 (VDD)
- new net I2C0.SCL: J23.1 (Pin_1), U28.4 (SCK)
- new net I2C0.SDA: J26.1 (Pin_1), U28.3 (SDI)
Other:
- note added: "Barometer DPS368 on I2C0, 0x76 (SDO to GND), I2C mode (CSB to VDDIO). Pull-ups R11/R12 to +3.3V. Betaflight: baro_hardware DPS310."
- note added: "D10: flyback for a magnetic 5 V buzzer on J29/J33 (Q1 AP1606 is 20 V)."
- note added: "I2C out"
- title: (none) -> Pads
