File: hardware/fc_power.kicad_sch (KiCad schematic)
At the start: 25 parts, among them U8 LMR51430YFDDCR, U9 LMR51430YFDDCR

Commit message: schematic review: USB D+/D- swap, bulk cap parts, VTX UART, EN series R, density cuts, ERC cleanup, docs (#24)
Items 1, 2, 3, 5, 8, 9, 10, 11, 12, 13, 14 (partial), 17, 18, 19, 20, 21, 22, 23, 6.
Edits are structured s-expression edits re-saved by kicad-cli sch upgrade.

Co-authored-by: Stan <stan@openaio.local>
Co-authored-by: Claude Opus 5.5 <noreply@anthropic.com>
Parts:
- removed D5: LED_1_Green, LED_SMD:LED_0402_1005Metric, symbol Device:LED
- removed R16: 2.4k, Resistor_SMD:R_0201_0603Metric, symbol Device:R
- removed TP2: TestPoint, TestPoint:TestPoint_Pad_D1.0mm, symbol Connector:TestPoint
- added R96: 100k, Resistor_SMD:R_0201_0603Metric, symbol Device:R
- C35, C36: value C -> 4.7uF 50v; LCSC (none) -> C98192; MPN (none) -> CL21A475KBQNNNE; Manufacturer (none) -> Samsung Electro-Mechanics
- C39, C40: value C -> 10uF 50V; LCSC (none) -> C89632; MPN (none) -> CL31B106KBHNNNE; Manufacturer (none) -> Samsung Electro-Mechanics
- R12: MPN (none) -> AF0201FR-076K49L; Manufacturer (none) -> YAGEO
- R15: MPN (none) -> RC0201FR-077K5L; Manufacturer (none) -> YAGEO
- U8, U9: symbol lib:LMR51420YDDCR -> OpenDrone:LMR51430YFDDCR
Connections:
- net 10V_ENABLE: now also R96.1; no longer U8.5 (EN)
- new net: R96.2, U8.5 (EN)
