File: hardware/fc_power.kicad_sch (KiCad schematic)
At the start: 25 parts, among them U8 LMR51430YFDDCR, U9 LMR51430YFDDCR

Commit message: One board: Base + Core merged on the 8L HDI stackup, replaces the OpenFC-Core module layout (#25)
* Base fully routed (recovered from KiCad local history, 2026-08-22)

The finished Base route was never committed: the last Base commit (ce0aa59)
had 57 unconnected. Recovered from hardware/.history snapshot 55d048e
(last save 2026-08-22 15:03), on top of ce0aa59.

DRC (kicad-cli 10):
- Base: 0 unconnected, 0 shorts, 6 errors (3 x U23 own pad-to-pad
  clearance, USB1 NPTH: 1 clearance + 2 annular width), 111 warnings
- Core: 0 unconnected, 0 errors

Co-Authored-By: Claude Opus 5.5 <noreply@anthropic.com>

* Power: +10V buck always on with battery, 10V_ENABLE removed

CIRCUIT_REVIEW B1: the LMR51430 +10V buck U3 (NSG2065Q gate drive and VTX power) was enabled by RP2354A GPIO27 over LGA pad 1 with no pull, so firmware or a Betaflight PINIO could cut ESC gate drive, and on USB-only power a high GPIO27 drove EN with VIN = 0, which the LMR51430 datasheet forbids. U3 EN is now tied to +BATT exactly like U4 (datasheet: EN may be tied to VIN; no parts added). Base: U3.5 keeps its B.Cu stub and through via, re-netted to +BATT so the via lands in the +BATT planes; the In2 run, the via and the F.Cu stub to J90 pad 1 are removed. Core: the GPIO27 route to J91 pad 1 is removed. LGA pad 1 and GPIO27 are free (no-connect); the root marker TP14 of the old net is dropped. Boards saved by pcbnew 10.0.6 without zone refill; the "Tokyo" silkscreen render caches were re-rendered with a substitute font (Tokyo not installed here).

Co-Authored-By: Claude Opus 5.5 <noreply@anthropic.com>
Claude-Session: https://claude.ai/code/session_01KTp3FLjVXfXdWrkmr6af7d

* Review of the split Core/Base design, NextPCB rules, re-route plan

Circuit review against datasheets, layout review (LGA interface, DC power
solver, noise, density, assembly, DRC) with the scripts that produced every
number, NextPCB fab and assembly limits with sources, and the plan with the
decisions taken for the re-route.

Co-Author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
Parts:
- added C107, C116: 100nF, lib:C_0402_1005Metric, symbol Device:C
- added C110, C111: 1uF, lib:C_0201_0603Metric, symbol Device:C
- added C112, C113: 22uF, lib:C_0603_1608Metric, symbol Device:C
- added C25, C27: 4.7uF, lib:C_0402_1005Metric, symbol Device:C
- added C26, C28: 1uF, lib:C_0402_1005Metric, symbol Device:C
- added D6, D7: LED_1_Green, lib:LED_0402_1005Metric, symbol Device:LED
- added R23: 6.49k, lib:R_0201_0603Metric, symbol Device:R
- added R24: 510R, lib:R_0201_0603Metric, symbol Device:R
- added U27: TLV75533PDQNR, lib:X2SON-4_L1.0-W1.0-P0.65-TL-EP, symbol lib:TLV75533PDQNR
- added U6: LP5912-1.8DRVR, lib:WSON-6-1EP_2x2mm_P0.65mm_EP1x1.6mm_ThermalVias, symbol lib:LP5912-1.8DRVR
- added U7: LP5912-3.3DRVR, lib:WSON-6-1EP_2x2mm_P0.65mm_EP1x1.6mm, symbol lib:LP5912-3.3DRV_1
- C102: renamed from C35; value C -> 4.7uF 50v; footprint Capacitor_SMD:C_0805_2012Metric -> lib:C_0805_2012Metric; LCSC (none) -> C98192; MPN (none) -> CL21A475KBQNNNE; Manufacturer (none) -> Samsung Electro-Mechanics
- C103: renamed from C36; value C -> 4.7uF 50v; footprint Capacitor_SMD:C_0805_2012Metric -> lib:C_0805_2012Metric; LCSC (none) -> C98192; MPN (none) -> CL21A475KBQNNNE; Manufacturer (none) -> Samsung Electro-Mechanics
- C105: renamed from C39; value C -> 4.7uF 50v; footprint Capacitor_SMD:C_1206_3216Metric -> lib:C_1206_3216Metric; LCSC (none) -> C380366; MPN (none) -> TCC1206X7R475K500HT; Manufacturer (none) -> CCTC
- C106: renamed from C40; value C -> 4.7uF 50v; footprint Capacitor_SMD:C_1206_3216Metric -> lib:C_1206_3216Metric; LCSC (none) -> C380366; MPN (none) -> TCC1206X7R475K500HT; Manufacturer (none) -> CCTC
- C18: renamed from C33; footprint Capacitor_SMD:C_0805_2012Metric -> lib:C_0805_2012Metric
- C19: renamed from C34; footprint Capacitor_SMD:C_0805_2012Metric -> lib:C_0805_2012Metric
- C20: renamed from C37; footprint Capacitor_SMD:C_0201_0603Metric -> lib:C_0201_0603Metric
- C21: renamed from C38; footprint Capacitor_SMD:C_0201_0603Metric -> lib:C_0201_0603Metric
- C23: renamed from C41; footprint Capacitor_SMD:C_0603_1608Metric -> lib:C_0603_1608Metric
- C24: renamed from C42; footprint Capacitor_SMD:C_0603_1608Metric -> lib:C_0603_1608Metric
- D4, D5: footprint LED_SMD:LED_0402_1005Metric -> lib:LED_0402_1005Metric; MPN XL-1005UGC -> XL-1005UGC
- R17: renamed from R11; footprint Resistor_SMD:R_0201_0603Metric -> lib:R_0201_0603Metric
- R18: renamed from R12; footprint Resistor_SMD:R_0201_0603Metric -> lib:R_0201_0603Metric; MPN (none) -> AF0201FR-076K49L; Manufacturer (none) -> YAGEO
- R19: renamed from R13; footprint Resistor_SMD:R_0201_0603Metric -> lib:R_0201_0603Metric
- R20: renamed from R14; footprint Resistor_SMD:R_0201_0603Metric -> lib:R_0201_0603Metric
- R21: renamed from R15; footprint Resistor_SMD:R_0201_0603Metric -> lib:R_0201_0603Metric; MPN (none) -> RC0201FR-077K5L; Manufacturer (none) -> YAGEO
- R22: renamed from R16; footprint Resistor_SMD:R_0201_0603Metric -> lib:R_0201_0603Metric; MPN (none) -> RTT012401FTH; Manufacturer (none) -> RALEC
- TP30: renamed from TP2; footprint TestPoint:TestPoint_Pad_D1.0mm -> lib:TestPoint_Pad_D1.0mm
- renumbered L6 to L2, L7 to L3, U8 to U3, U9 to U4
Connections:
- net 10V_ENABLE is gone; now on net +BATT: U3.5 (EN)
- net +10V: now also C112.1, C113.1
- net +4v5: now also C25.1, C26.1, R23.1, U6.4 (EN), U6.6 (IN), U7.4 (EN), U7.6 (IN)
- net +5V: now also C110.1, U27.3 (EN), U27.4 (IN)
- net +BATT: now also C107.1, C116.1
- net GND: now also C107.2, C110.2, C111.2, C112.2, C113.2, C116.2, C25.2, C26.2, C27.2, C28.2, D6.1 (K), D7.1 (K), U27.2 (GND), U27.5 (EP), U6.5 (GND), U6.7 (EP), U7.3 (PG), U7.5 (GND), U7.7 (EP)
- new net: D6.2 (A), R24.2
- new net +1.8V_GYRO: C27.1, U6.1 (OUT)
- new net +3.3V: C28.1, U7.1 (OUT)
- new net +3V3: R24.1
- new net +3V3_ESC: C111.1, U27.1 (OUT)
- new net 1.8V_PG: D7.2 (A), R23.2, U6.3 (PG)
- no-connect marks 0 -> 1
Other:
- note added: "+10V output caps C112, C113 (with C23 at U3, Base B side)"
- note added: "1.8V LDO for IMU (high PSRR)"
- note added: "3.3V 0.5A MAIN LDO"
- note added: "3.3V ESC MCU LDO (battery only, +5V buck) AT32F421 VDD/VDDA off on USB-only power"
- note added: "C116: 0.1 uF at U3 VIN pins 3/5 (LMR51430 9.2.2.6), next to the pins."
- note added: "Up to 6.5V input (5V) Thermal Protection Short circuit protection Reverse current protection Low noise for RF and analog circuits"
- title: (none) -> Power
