File: hardware/rx_esp32c3_sx1281.kicad_sch (KiCad schematic)
At the start: 43 parts, among them U19 SX1281IMLTRT, U20 ESP32-C3, U21 TLV75533PDQNR, X2 CJ17-400001010B20

Commit message: One board: Base + Core merged on the 8L HDI stackup, replaces the OpenFC-Core module layout (#25)
* Base fully routed (recovered from KiCad local history, 2026-08-22)

The finished Base route was never committed: the last Base commit (ce0aa59)
had 57 unconnected. Recovered from hardware/.history snapshot 55d048e
(last save 2026-08-22 15:03), on top of ce0aa59.

DRC (kicad-cli 10):
- Base: 0 unconnected, 0 shorts, 6 errors (3 x U23 own pad-to-pad
  clearance, USB1 NPTH: 1 clearance + 2 annular width), 111 warnings
- Core: 0 unconnected, 0 errors

Co-Authored-By: Claude Opus 5.5 <noreply@anthropic.com>

* Power: +10V buck always on with battery, 10V_ENABLE removed

CIRCUIT_REVIEW B1: the LMR51430 +10V buck U3 (NSG2065Q gate drive and VTX power) was enabled by RP2354A GPIO27 over LGA pad 1 with no pull, so firmware or a Betaflight PINIO could cut ESC gate drive, and on USB-only power a high GPIO27 drove EN with VIN = 0, which the LMR51430 datasheet forbids. U3 EN is now tied to +BATT exactly like U4 (datasheet: EN may be tied to VIN; no parts added). Base: U3.5 keeps its B.Cu stub and through via, re-netted to +BATT so the via lands in the +BATT planes; the In2 run, the via and the F.Cu stub to J90 pad 1 are removed. Core: the GPIO27 route to J91 pad 1 is removed. LGA pad 1 and GPIO27 are free (no-connect); the root marker TP14 of the old net is dropped. Boards saved by pcbnew 10.0.6 without zone refill; the "Tokyo" silkscreen render caches were re-rendered with a substitute font (Tokyo not installed here).

Co-Authored-By: Claude Opus 5.5 <noreply@anthropic.com>
Claude-Session: https://claude.ai/code/session_01KTp3FLjVXfXdWrkmr6af7d

* Review of the split Core/Base design, NextPCB rules, re-route plan

Circuit review against datasheets, layout review (LGA interface, DC power
solver, noise, density, assembly, DRC) with the scripts that produced every
number, NextPCB fab and assembly limits with sources, and the plan with the
decisions taken for the re-route.

Co-Author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
Parts:
- AE1: renamed from AE2; footprint OpenRX-Shared:ANT-SMD_L3.2-W1.6 -> lib:ANT-SMD_L3.2-W1.6; symbol OpenRX-Shared:2450AT18A100E -> lib:2450AT18A100E; MPN (none) -> 2450AT18A100E; Manufacturer (none) -> JOHANSON(约翰逊)
- C1: renamed from C90; footprint Capacitor_SMD:C_0201_0603Metric -> lib:C_0201_0603Metric; MPN (none) -> GRM0335C1H150JA01D; Manufacturer (none) -> Murata Electronics
- C10: renamed from C103; footprint Capacitor_SMD:C_0201_0603Metric -> lib:C_0201_0603Metric; MPN (none) -> GRM033R61A105ME44D; Manufacturer (none) -> Murata Electronics
- C11: renamed from C93; footprint Capacitor_SMD:C_0402_1005Metric -> lib:C_0402_1005Metric; MPN (none) -> GRM155R60J106ME44D; Manufacturer (none) -> Murata Electronics
- C12: renamed from C84; footprint Capacitor_SMD:C_0201_0603Metric -> lib:C_0201_0603Metric; MPN (none) -> GRM033R61E104KE14D; Manufacturer (none) -> Murata Electronics
- C13: renamed from C83; footprint Capacitor_SMD:C_0201_0603Metric -> lib:C_0201_0603Metric; MPN (none) -> GRM033R61E104KE14D; Manufacturer (none) -> Murata Electronics
- C14: renamed from C88; footprint Capacitor_SMD:C_0201_0603Metric -> lib:C_0201_0603Metric; MPN (none) -> GRM033R61E104KE14D; Manufacturer (none) -> Murata Electronics
- C15: renamed from C104; footprint Capacitor_SMD:C_0201_0603Metric -> lib:C_0201_0603Metric; MPN (none) -> GRM033R61A105ME44D; Manufacturer (none) -> Murata Electronics
- C16: renamed from C106; footprint Capacitor_SMD:C_0402_1005Metric -> lib:C_0402_1005Metric; MPN (none) -> CL05A106MQ5NUNC; Manufacturer (none) -> Samsung Electro-Mechanics
- C17: renamed from C89; footprint Capacitor_SMD:C_0201_0603Metric -> lib:C_0201_0603Metric; MPN (none) -> GRM033R61E104KE14D; Manufacturer (none) -> Murata Electronics
- C19: renamed from C87; footprint Capacitor_SMD:C_0201_0603Metric -> lib:C_0201_0603Metric; MPN (none) -> 0201B102K500NT; Manufacturer (none) -> FH (Guangdong Fenghua)
- C20: renamed from C86; footprint Capacitor_SMD:C_0201_0603Metric -> lib:C_0201_0603Metric; MPN (none) -> GRM033R60J474KE90D; Manufacturer (none) -> Murata Electronics
- C21: renamed from C107; footprint Capacitor_SMD:C_0201_0603Metric -> lib:C_0201_0603Metric; MPN (none) -> GRM0335C1H1R2BA01D; Manufacturer (none) -> Murata Electronics
- C22: renamed from C105; footprint Capacitor_SMD:C_0201_0603Metric -> lib:C_0201_0603Metric; MPN (none) -> GRM0335C1H1R2BA01D; Manufacturer (none) -> Murata Electronics
- C23: renamed from C99; footprint Capacitor_SMD:C_0201_0603Metric -> lib:C_0201_0603Metric; MPN (none) -> GRM033R61A105ME44D; Manufacturer (none) -> Murata Electronics
- C24: renamed from C98; footprint Capacitor_SMD:C_0201_0603Metric -> lib:C_0201_0603Metric; MPN (none) -> GRM033R61A103KA01J; Manufacturer (none) -> Murata Electronics
- C25: renamed from C95; footprint Capacitor_SMD:C_0201_0603Metric -> lib:C_0201_0603Metric; MPN (none) -> GRM033R61A105ME44D; Manufacturer (none) -> Murata Electronics
- C26: renamed from C85; footprint Capacitor_SMD:C_0201_0603Metric -> lib:C_0201_0603Metric; MPN (none) -> GRM033R61A103KA01J; Manufacturer (none) -> Murata Electronics
- C27: renamed from C91; footprint Capacitor_SMD:C_0201_0603Metric -> lib:C_0201_0603Metric; MPN (none) -> GRM033R61A103KA01J; Manufacturer (none) -> Murata Electronics
- C28: renamed from C102; footprint Capacitor_SMD:C_0201_0603Metric -> lib:C_0201_0603Metric; MPN (none) -> GRM033R61A105ME44D; Manufacturer (none) -> Murata Electronics
- C3: renamed from C92; footprint Capacitor_SMD:C_0201_0603Metric -> lib:C_0201_0603Metric; MPN (none) -> GRM0335C1H150JA01D; Manufacturer (none) -> Murata Electronics
- C4: renamed from C101; footprint Capacitor_SMD:C_0201_0603Metric -> lib:C_0201_0603Metric; MPN (none) -> GRM033R61A105ME44D; Manufacturer (none) -> Murata Electronics
- C5: renamed from C96; footprint Capacitor_SMD:C_0201_0603Metric -> lib:C_0201_0603Metric; MPN (none) -> GRM033R61E104KE14D; Manufacturer (none) -> Murata Electronics
- C6: renamed from C97; footprint Capacitor_SMD:C_0201_0603Metric -> lib:C_0201_0603Metric; MPN (none) -> GRM033R61E104KE14D; Manufacturer (none) -> Murata Electronics
- C8: renamed from C100; footprint Capacitor_SMD:C_0402_1005Metric -> lib:C_0402_1005Metric; MPN (none) -> CL05A106MQ5NUNC; Manufacturer (none) -> Samsung Electro-Mechanics
- C9: renamed from C94; footprint Capacitor_SMD:C_0201_0603Metric -> lib:C_0201_0603Metric; MPN (none) -> GRM033R61E104KE14D; Manufacturer (none) -> Murata Electronics
- D1: renamed from D6; footprint OpenRX-Shared:LED-SMD_4P-L1.0-W1.0-TL_XL-1010RGBC-WS2812B -> lib:LED-SMD_4P-L1.0-W1.0-TL_XL-1010RGBC-WS2812B; symbol OpenRX-Shared:XL-1010RGBC-WS2812B -> lib:XL-1010RGBC-WS2812B; LCSC (none) -> C5349953; MPN (none) -> XL-1010RGBC-2812B; Manufacturer (none) -> XINGLIGHT
- FL1: renamed from FL2; footprint OpenRX-Shared:FILTER-SMD_4P-L1.0-W0.5-L -> lib:FILTER-SMD_4P-L1.0-W0.5-L; symbol OpenRX-Shared:2450FM07D0034T -> lib:2450FM07D0034T
- JP1: footprint OpenDrone:RF-SMD_FRF05002-JSS103M -> lib:RF-SMD_FRF05002-JSS103M; symbol OpenDrone:U.FL-R-SMT-1(80) -> lib:U.FL-R-SMT-1(80); MPN (none) -> U.FL-R-SMT-1(80); Manufacturer (none) -> Hirose
- L1: renamed from L9; footprint Inductor_SMD:L_0201_0603Metric -> lib:L_0201_0603Metric; MPN (none) -> LQP03TN24NH02D; Manufacturer (none) -> Murata Electronics
- L2: renamed from L11; footprint Inductor_SMD:L_0201_0603Metric -> lib:L_0201_0603Metric; MPN (none) -> LQP03TN2N5C02D; Manufacturer (none) -> Murata Electronics
- L3: renamed from L10; footprint Inductor_SMD:L_0201_0603Metric -> lib:L_0201_0603Metric; MPN (none) -> LQP03TN2N0B02D; Manufacturer (none) -> Murata Electronics
- L4: renamed from L8; footprint Inductor_SMD:L_0805_2012Metric -> lib:L_0805_2012Metric; LCSC (none) -> C383402; MPN (none) -> MLZ2012M150WT000; Manufacturer (none) -> TDK
- OSC1: renamed from OSC2; footprint OpenRX-Shared:OSC-SMD_4P-L2.0-W1.6-BL_TXC_7Z -> lib:OSC-SMD_4P-L2.0-W1.6-BL_TXC_7Z; symbol OpenRX-Shared:OW7EL89CENUNFAYLC-52M -> lib:OW7EL89CENUNFAYLC-52M; MPN (none) -> OW7EL89CENUNFAYLC-52M; Manufacturer (none) -> TXC
- R2: renamed from R93; footprint Resistor_SMD:R_0201_0603Metric -> lib:R_0201_0603Metric; MPN (none) -> RC0201FR-0710KL; Manufacturer (none) -> YAGEO
- R3: renamed from R94; footprint Resistor_SMD:R_0201_0603Metric -> lib:R_0201_0603Metric; MPN (none) -> RC0201FR-0710KL; Manufacturer (none) -> YAGEO
- R4: renamed from R95; footprint Resistor_SMD:R_0201_0603Metric -> lib:R_0201_0603Metric; MPN (none) -> RC0201FR-0710KL; Manufacturer (none) -> YAGEO
- R5: renamed from R96; footprint Resistor_SMD:R_0201_0603Metric -> lib:R_0201_0603Metric; MPN (none) -> RC0201FR-0710KL; Manufacturer (none) -> YAGEO
- TP5: renamed from TP11; footprint OpenRX-Shared:SolderPad_1.2x2.0mm -> lib:SolderPad_1.2x2.0mm; now left out of the parts list
- U1: renamed from U20; value ESP32-C3 -> ESP32-C3FH4; footprint Package_DFN_QFN:QFN-32-1EP_5x5mm_P0.5mm_EP3.7x3.7mm -> lib:QFN-32-1EP_5x5mm_P0.5mm_EP3.7x3.7mm; LCSC (none) -> C2858491; MPN (none) -> ESP32-C3FH4; Manufacturer (none) -> Espressif Systems
- U2: renamed from U21; footprint OpenRX-Shared:X2SON-4_L1.0-W1.0-P0.65-TL-EP -> lib:X2SON-4_L1.0-W1.0-P0.65-TL-EP; symbol OpenRX-Shared:TLV75533PDQNR -> lib:TLV75533PDQNR; MPN (none) -> TLV75533PDQNR; Manufacturer (none) -> Texas Instruments
- U3: renamed from U19; footprint OpenRX-Shared:QFN-24_L4.0-W4.0-P0.50-TL-EP2.6 -> lib:QFN-24_L4.0-W4.0-P0.50-TL-EP2.6; symbol OpenRX-Shared:SX1281IMLTRT -> lib:SX1281IMLTRT; MPN (none) -> SX1281IMLTRT; Manufacturer (none) -> Semtech
- X1: renamed from X2; footprint OpenRX-Shared:CRYSTAL-SMD_4P-L1.6-W1.2-BL -> lib:CRYSTAL-SMD_4P-L1.6-W1.2-BL; symbol OpenRX-Shared:CJ17-400001010B20 -> lib:CJ17-400001010B20; MPN (none) -> CJ17-400001010B20; Manufacturer (none) -> Jiangsu Changjing Electronics
Connections:
- net +3V3: no longer D1.2 (VDD)
- net +4v5: now also D1.2 (VDD)
- net GND: now also U3.5 (GND)
- no-connect marks 15 -> 14
